Commit message: Tweak lenghts

File: src/xarm_description/urdf/xarm.urdf (robot description, URDF)
Before this commit: robot xarm, 6 links, 5 joints
Joints:
- joint xarm_3_joint: origin xyz=0 0.0 0.09825 rpy=0 0 0 -> xyz=0 0.0 0.098 rpy=0 0 0
- joint xarm_4_joint: origin xyz=0 0.0 0.09765 rpy=0 0 0 -> xyz=0 0.0 0.098 rpy=0 0 0
